File: 555_Timer_Clock.kicad_sch (KiCad schematic)
At the start: 16 parts, among them J1 +5V, J2 CLK_Out, SW1 Trigger, SW2 RST, U1 ICM7555xB

Commit message: Update PCB with connections
Parts:
- J1: footprint (none) -> my_footprints:Terminal_Block_5mm
- SW1: footprint (none) -> my_footprints:slide_switch_2.54mm
- SW2: footprint (none) -> my_footprints:tact_switch_5mm
Changed lines of the file:
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@@
 		)
 		(instances
-			(project ""
+			(project "555_Timer_Clock"
 				(path "/20801574-c7e9-4deb-947a-5143e918b622"
 					(reference "J2")
@@
 		)
 		(instances
-			(project ""
+			(project "555_Timer_Clock"
 				(path "/20801574-c7e9-4deb-947a-5143e918b622"
 					(reference "H2")
@@
 			)
 		)
-		(property "Footprint" ""
+		(property "Footprint" "my_footprints:Terminal_Block_5mm"
 			(at 161.29 97.79 0)
 			(effects
@@
 		)
 		(instances
-			(project ""
+			(project "555_Timer_Clock"
 				(path "/20801574-c7e9-4deb-947a-5143e918b622"
 					(reference "J1")
@@
 		)
 		(instances
-			(project ""
+			(project "555_Timer_Clock"
 				(path "/20801574-c7e9-4deb-947a-5143e918b622"
 					(reference "#FLG02")
@@
 		)
 		(instances
-			(project ""
+			(project "555_Timer_Clock"
 				(path "/20801574-c7e9-4deb-947a-5143e918b622"
 					(reference "C2")
@@
 			)
 		)
-		(property "Footprint" ""
+		(property "Footprint" "my_footprints:tact_switch_5mm"
 			(at 160.02 82.55 0)
 			(effects
@@
 		)
 		(instances
-			(project ""
+			(project "555_Timer_Clock"
 				(path "/20801574-c7e9-4deb-947a-5143e918b622"
 					(reference "SW2")
@@
 		)
 		(instances
-			(project ""
+			(project "555_Timer_Clock"
 				(path "/20801574-c7e9-4deb-947a-5143e918b622"
 					(reference "D1")
@@
 		)
 		(instances
-			(project ""
+			(project "555_Timer_Clock"
 				(path "/20801574-c7e9-4deb-947a-5143e918b622"
 					(reference "H1")
@@
 		)
 		(instances
-			(project ""
+			(project "555_Timer_Clock"
 				(path "/20801574-c7e9-4deb-947a-5143e918b622"
 					(reference "R1")
@@
 		)
 		(instances
-			(project ""
+			(project "555_Timer_Clock"
 				(path "/20801574-c7e9-4deb-947a-5143e918b622"
 					(reference "C1")
@@
 		)
 		(instances
-			(project ""
+			(project "555_Timer_Clock"
 				(path "/20801574-c7e9-4deb-947a-5143e918b622"
 					(reference "H3")
@@
 		)
 		(instances
-			(project ""
+			(project "555_Timer_Clock"
 				(path "/20801574-c7e9-4deb-947a-5143e918b622"
 					(reference "U1")
@@
 		)
 		(instances
-			(project ""
+			(project "555_Timer_Clock"
 				(path "/20801574-c7e9-4deb-947a-5143e918b622"
 					(reference "H4")
@@
 		)
 		(instances
-			(project ""
+			(project "555_Timer_Clock"
 				(path "/20801574-c7e9-4deb-947a-5143e918b622"
 					(reference "#PWR01")
@@
 		)
 		(instances
-			(project ""
+			(project "555_Timer_Clock"
 				(path "/20801574-c7e9-4deb-947a-5143e918b622"
 					(reference "R4")
@@
 			)
 		)
-		(property "Footprint" ""
+		(property "Footprint" "my_footprints:slide_switch_2.54mm"
 			(at 160.02 74.93 0)
 			(effects
@@
 		)
 		(instances
-			(project ""
+			(project "555_Timer_Clock"
 				(path "/20801574-c7e9-4deb-947a-5143e918b622"
 					(reference "SW1")
